Commit message: 6.4.2

File: chapt6/chapt6_ws/src/fishbot_description/urdf/fishbot/actuator/caster.urdf.xacro (robot description, xacro)
@@ -1,9 +1,10 @@
 <?xml version="1.0"?>
 <robot xmlns:xacro="http://www.ros.org/wiki/xacro">
+    <xacro:include filename="$(find fishbot_description)/urdf/fishbot/common_inertia.xacro"/>
     <xacro:macro name="caster_xacro" params="caster_name xyz rpy">
         <!-- 机器的万向轮 -->
         <link name="${caster_name}_link">
         <!-- 部件的外观描述 -->
-            <visual>
+            <visual name="caster_visual">
             <!-- 沿着自己几何中心的偏移和旋转量 -->
                 <origin xyz="0.0 0.0 0.0" rpy="0.0 0.0 0.0"/>
@@ -15,4 +16,16 @@
                 </material>
             </visual>
+            <!-- 碰撞属性 -->
+            <collision name="caster_collision">
+             <!-- 沿着自己几何中心的偏移和旋转量 -->
+                <origin xyz="0.0 0.0 0.0" rpy="0.0 0.0 0.0"/>
+                <geometry>
+                    <sphere radius="0.016"/>
+                </geometry>
+                <material name="yellow">
+                    <color rgba="1.0 1.0 0.0 0.8"/>
+                </material>
+            </collision>
+            <xacro:sphere_inertia m="0.01" r="0.016" />
         </link>
         <!-- 机器人的关节，用于连接caster_link和base_link -->

File: chapt6/chapt6_ws/src/fishbot_description/urdf/fishbot/actuator/wheel.urdf.xacro (robot description, xacro)
@@ -1,9 +1,10 @@
 <?xml version="1.0"?>
 <robot xmlns:xacro="http://www.ros.org/wiki/xacro">
+    <xacro:include filename="$(find fishbot_description)/urdf/fishbot/common_inertia.xacro"/>
     <xacro:macro name="wheel_xacro" params="wheel_name xyz rpy">
         <!-- 机器的wheel -->
         <link name="${wheel_name}_link">
         <!-- 部件的外观描述 -->
-            <visual>
+            <visual name="wheel_visual">
             <!-- 沿着自己几何中心的偏移和旋转量 -->
                 <origin xyz="0.0 0.0 0.0" rpy="1.57079 0.0 0.0"/>
@@ -15,4 +16,15 @@
                 </material>
             </visual>
+            <collision name="wheel_collision">
+            <!-- 沿着自己几何中心的偏移和旋转量 -->
+                <origin xyz="0.0 0.0 0.0" rpy="1.57079 0.0 0.0"/>
+                <geometry>
+                    <cylinder radius="0.032" length="0.04"/>
+                </geometry>
+                <material name="yellow">
+                    <color rgba="1.0 1.0 0.0 0.8"/>
+                </material>
+            </collision>
+            <xacro:cylinder_inertia m="0.1" h="0.04" r="0.032"/>
         </link>
         <!-- 机器人的关节，用于连接wheel_link和base_link -->

File: chapt6/chapt6_ws/src/fishbot_description/urdf/fishbot/base.urdf.xacro (robot description, xacro)
@@ -1,4 +1,5 @@
 <?xml version="1.0"?>
 <robot xmlns:xacro="http://www.ros.org/wiki/xacro">
+    <xacro:include filename="$(find fishbot_description)/urdf/fishbot/common_inertia.xacro"/>
     <xacro:macro name="base_xacro" params="length radius">
         <link name="base_footprint" />
@@ -6,5 +7,5 @@
         <link name="base_link">
             <!-- 部件的外观描述 -->
-            <visual>
+            <visual name="base_visual">
                 <!-- 沿着自己几何中心的偏移和旋转量 -->
                 <origin xyz="0.0 0.0 0.0" rpy="0.0 0.0 0.0"/>
@@ -19,4 +20,19 @@
                 </material>
             </visual>
+            <!-- 部件的碰撞描述 -->
+            <collision name="base_collision">
+                <!-- 沿着自己几何中心的偏移和旋转量 -->
+                <origin xyz="0.0 0.0 0.0" rpy="0.0 0.0 0.0"/>
+                <!-- 几何形状 -->
+                <geometry>
+                    <!-- 圆柱体 -->
+                    <cylinder radius="${radius}" length="${length}"/>
+                </geometry>
+                <!-- 材料颜色 -->
+                <material name="white">
+                    <color rgba="1.0 1.0 1.0 0.5"/>
+                </material>
+            </collision>
+            <xacro:cylinder_inertia m="1.0" r="${radius}" h="${length}" />
         </link>
         <joint name="base_joint" type="fixed">

File: chapt6/chapt6_ws/src/fishbot_description/urdf/fishbot/sensor/camera.urdf.xacro (robot description, xacro)
@@ -1,9 +1,10 @@
 <?xml version="1.0"?>
 <robot xmlns:xacro="http://www.ros.org/wiki/xacro">
+    <xacro:include filename="$(find fishbot_description)/urdf/fishbot/common_inertia.xacro"/>
     <xacro:macro name="camera_xacro" params="camera_name xyz rpy">
         <!-- 机器的摄像头 -->
         <link name="${camera_name}_link">
         <!-- 部件的外观描述 -->
-            <visual>
+            <visual name="camera_visual">
             <!-- 沿着自己几何中心的偏移和旋转量 -->
                 <origin xyz="0.0 0.0 0.0" rpy="0.0 0.0 0.0"/>
@@ -15,4 +16,15 @@
                 </material>
             </visual>
+            <collision name="camera_collision">
+            <!-- 沿着自己几何中心的偏移和旋转量 -->
+                <origin xyz="0.0 0.0 0.0" rpy="0.0 0.0 0.0"/>
+                <geometry>
+                    <box size="0.02 0.10 0.02"/>
+                </geometry>
+                <material name="blue">
+                    <color rgba="0.0 0.0 1.0 0.5"/>
+                </material>
+            </collision>
+            <xacro:box_inertia m="0.01" w="0.02" h="0.10" d="0.02" />
         </link>
         <!-- 机器人的关节，用于连接camera_link和base_link -->

File: chapt6/chapt6_ws/src/fishbot_description/urdf/fishbot/sensor/imu.urdf.xacro (robot description, xacro)
@@ -1,9 +1,10 @@
 <?xml version="1.0"?>
 <robot xmlns:xacro="http://www.ros.org/wiki/xacro">
+    <xacro:include filename="$(find fishbot_description)/urdf/fishbot/common_inertia.xacro"/>
     <xacro:macro name="imu_xacro" params="imu_name xyz rpy">
         <!-- 机器的imu -->
         <link name="${imu_name}_link">
         <!-- 部件的外观描述 -->
-            <visual>
+            <visual name="imu_visual">
             <!-- 沿着自己几何中心的偏移和旋转量 -->
                 <origin xyz="0.0 0.0 0.0" rpy="0.0 0.0 0.0"/>
@@ -15,4 +16,16 @@
                 </material>
             </visual>
+            <!-- 部件的碰撞描述 -->
+            <collision name="imu_collision">
+            <!-- 沿着自己几何中心的偏移和旋转量 -->
+                <origin xyz="0.0 0.0 0.0" rpy="0.0 0.0 0.0"/>
+                <geometry>
+                    <box size="0.02 0.02 0.02"/>
+                </geometry>
+                <material name="blue">
+                    <color rgba="0.0 0.0 1.0 0.5"/>
+                </material>
+            </collision>
+            <xacro:box_inertia m="0.01" w="0.02" d="0.02" h="0.02"/>
         </link>
         <!-- 机器人的关节，用于连接imu_link和base_link -->

File: chapt6/chapt6_ws/src/fishbot_description/urdf/fishbot/sensor/laser.urdf.xacro (robot description, xacro)
@@ -1,8 +1,9 @@
 <?xml version="1.0"?>
 <robot xmlns:xacro="http://www.ros.org/wiki/xacro">
+    <xacro:include filename="$(find fishbot_description)/urdf/fishbot/common_inertia.xacro"/>
     <xacro:macro name="laser_xacro" params="laser_name xyz rpy">
         <!-- 雷达支撑杆 laser_cylinder_link -->
         <link name="${laser_name}_cylinder_link">
-            <visual>
+            <visual name="laser_cylinder_visual">
                 <origin xyz="0.0 0.0 0.0" rpy="0.0 0.0 0.0"/>
                 <geometry>
@@ -13,9 +14,19 @@
                 </material>
             </visual>
+            <collision name="laser_cylinder_collision">
+                <origin xyz="0.0 0.0 0.0" rpy="0.0 0.0 0.0"/>
+                <geometry>
+                    <cylinder radius="0.01" length="0.1"/>
+                </geometry>
+                <material name="gray">
+                    <color rgba="0.5 0.5 0.5 1.0"/>
+                </material>
+            </collision>
+            <xacro:cylinder_inertia m="0.01" r="0.01" h="0.10" />
         </link>
         <!-- 机器的激光雷达 -->
         <link name="${laser_name}_link">
         <!-- 部件的外观描述 -->
-            <visual>
+            <visual name="laser_visual">
             <!-- 沿着自己几何中心的偏移和旋转量 -->
                 <origin xyz="0.0 0.0 0.0" rpy="0.0 0.0 0.0"/>
@@ -27,4 +38,16 @@
                 </material>
             </visual>
+            <!-- 碰撞属性 -->
+            <collision name="laser_collision">
+            <!-- 沿着自己几何中心的偏移和旋转量 -->
+                <origin xyz="0.0 0.0 0.0" rpy="0.0 0.0 0.0"/>
+                <geometry>
+                    <cylinder radius="0.02" length="0.02"/>
+                </geometry>
+                <material name="blue">
+                    <color rgba="0.0 0.0 1.0 0.5"/>
+                </material>
+            </collision>
+            <xacro:cylinder_inertia m="0.03" r="0.02" h="0.02" />
         </link>
         <!-- 机器人的关节，用于连接laser_link和laser_cylinder_link -->

Commit message: 6.4

File: chapt6/chapt6_ws/src/fishbot_description/urdf/fishbot/actuator/caster.urdf.xacro (robot description, xacro)
@@ -3,8 +3,20 @@
     <xacro:include filename="$(find fishbot_description)/urdf/fishbot/common_inertia.xacro"/>
     <xacro:macro name="caster_xacro" params="caster_name xyz rpy">
+         <!-- gazebo中添加颜色 -->
+    <gazebo reference="${caster_name}_link">
+        <material>Gazebo/Yellow</material>
+        <!-- 切向摩擦系数 -->
+        <mu1 value="0.0" />
+        <!-- 法相摩擦系数 -->
+        <mu2 value="0.0" />
+        <!-- 接触刚度系数 -->
+        <kp value="1000000000.0" />
+        <!-- 阻尼系数 -->
+        <kd value="1.0" />
+    </gazebo>
         <!-- 机器的万向轮 -->
         <link name="${caster_name}_link">
         <!-- 部件的外观描述 -->
-            <visual name="caster_visual">
+            <visual>
             <!-- 沿着自己几何中心的偏移和旋转量 -->
                 <origin xyz="0.0 0.0 0.0" rpy="0.0 0.0 0.0"/>
@@ -17,5 +29,5 @@
             </visual>
             <!-- 碰撞属性 -->
-            <collision name="caster_collision">
+            <collision>
              <!-- 沿着自己几何中心的偏移和旋转量 -->
                 <origin xyz="0.0 0.0 0.0" rpy="0.0 0.0 0.0"/>

File: chapt6/chapt6_ws/src/fishbot_description/urdf/fishbot/actuator/wheel.urdf.xacro (robot description, xacro)
@@ -3,8 +3,20 @@
     <xacro:include filename="$(find fishbot_description)/urdf/fishbot/common_inertia.xacro"/>
     <xacro:macro name="wheel_xacro" params="wheel_name xyz rpy">
+     <!-- gazebo中添加颜色和摩擦系数 -->
+    <gazebo reference="${wheel_name}_link">
+        <material>Gazebo/Yellow</material>
+        <!-- 切向摩擦系数 -->
+        <mu1 value="20.0" />
+        <!-- 法相摩擦系数 -->
+        <mu2 value="20.0" />
+        <!-- 接触刚度系数 -->
+        <kp value="1000000000.0" />
+        <!-- 阻尼系数 -->
+        <kd value="1.0" />
+    </gazebo>
         <!-- 机器的wheel -->
         <link name="${wheel_name}_link">
         <!-- 部件的外观描述 -->
-            <visual name="wheel_visual">
+            <visual>
             <!-- 沿着自己几何中心的偏移和旋转量 -->
                 <origin xyz="0.0 0.0 0.0" rpy="1.57079 0.0 0.0"/>
@@ -16,5 +28,5 @@
                 </material>
             </visual>
-            <collision name="wheel_collision">
+            <collision>
             <!-- 沿着自己几何中心的偏移和旋转量 -->
                 <origin xyz="0.0 0.0 0.0" rpy="1.57079 0.0 0.0"/>

File: chapt6/chapt6_ws/src/fishbot_description/urdf/fishbot/base.urdf.xacro (robot description, xacro)
@@ -4,8 +4,12 @@
     <xacro:macro name="base_xacro" params="length radius">
         <link name="base_footprint" />
+     <!-- gazebo中添加颜色 -->
+    <gazebo reference="base_link">
+        <material>Gazebo/White</material>
+    </gazebo>
     <!-- 机器人的身体部分 -->
         <link name="base_link">
             <!-- 部件的外观描述 -->
-            <visual name="base_visual">
+            <visual>
                 <!-- 沿着自己几何中心的偏移和旋转量 -->
                 <origin xyz="0.0 0.0 0.0" rpy="0.0 0.0 0.0"/>
@@ -21,5 +25,5 @@
             </visual>
             <!-- 部件的碰撞描述 -->
-            <collision name="base_collision">
+            <collision>
                 <!-- 沿着自己几何中心的偏移和旋转量 -->
                 <origin xyz="0.0 0.0 0.0" rpy="0.0 0.0 0.0"/>

File: chapt6/chapt6_ws/src/fishbot_description/urdf/fishbot/fishbot.urdf.xacro (robot description, xacro)
@@ -18,4 +18,9 @@
 <xacro:caster_xacro caster_name="front_caster" xyz="0.08 0.0 -0.076" rpy="0.0 0.0 0.0"/>
 <xacro:caster_xacro caster_name="rear_caster" xyz="-0.08 0.0 -0.076" rpy="0.0 0.0 0.0"/>
+<!-- Gazebo 插件 -->
+<xacro:include filename="$(find fishbot_description)/urdf/fishbot/plugins/gazebo_control_plugin.xacro" />
+<xacro:gazebo_control_plugin />
+<!-- <xacro:include filename="$(find fishbot_description)/urdf/fishbot/fishbot.ros2_control.xacro" /> -->
+<!-- <xacro:fishbot_ros2_control /> -->
 </robot>
 <!-- ros2 launch fishbot_description display_robot.launch.py urdf_path:=/home/rick/ROS2_learn/chapt6/chapt6_ws/src/fishbot_description/urdf/fishbot/fishbot.urdf.xacro -->

File: chapt6/chapt6_ws/src/fishbot_description/urdf/fishbot/sensor/camera.urdf.xacro (robot description, xacro)
@@ -3,8 +3,12 @@
     <xacro:include filename="$(find fishbot_description)/urdf/fishbot/common_inertia.xacro"/>
     <xacro:macro name="camera_xacro" params="camera_name xyz rpy">
+    <!-- gazebo中添加颜色 -->
+    <gazebo reference="${camera_name}_link">
+        <material>Gazebo/Blue</material>
+    </gazebo>
         <!-- 机器的摄像头 -->
         <link name="${camera_name}_link">
         <!-- 部件的外观描述 -->
-            <visual name="camera_visual">
+            <visual>
             <!-- 沿着自己几何中心的偏移和旋转量 -->
                 <origin xyz="0.0 0.0 0.0" rpy="0.0 0.0 0.0"/>
@@ -16,5 +20,5 @@
                 </material>
             </visual>
-            <collision name="camera_collision">
+            <collision>
             <!-- 沿着自己几何中心的偏移和旋转量 -->
                 <origin xyz="0.0 0.0 0.0" rpy="0.0 0.0 0.0"/>

File: chapt6/chapt6_ws/src/fishbot_description/urdf/fishbot/sensor/imu.urdf.xacro (robot description, xacro)
@@ -3,8 +3,12 @@
     <xacro:include filename="$(find fishbot_description)/urdf/fishbot/common_inertia.xacro"/>
     <xacro:macro name="imu_xacro" params="imu_name xyz rpy">
+     <!-- gazebo中添加颜色 -->
+    <gazebo reference="${imu_name}_link">
+        <material>Gazebo/Blue</material>
+    </gazebo>
         <!-- 机器的imu -->
         <link name="${imu_name}_link">
         <!-- 部件的外观描述 -->
-            <visual name="imu_visual">
+            <visual>
             <!-- 沿着自己几何中心的偏移和旋转量 -->
                 <origin xyz="0.0 0.0 0.0" rpy="0.0 0.0 0.0"/>
@@ -17,5 +21,5 @@
             </visual>
             <!-- 部件的碰撞描述 -->
-            <collision name="imu_collision">
+            <collision>
             <!-- 沿着自己几何中心的偏移和旋转量 -->
                 <origin xyz="0.0 0.0 0.0" rpy="0.0 0.0 0.0"/>

File: chapt6/chapt6_ws/src/fishbot_description/urdf/fishbot/sensor/laser.urdf.xacro (robot description, xacro)
@@ -3,7 +3,14 @@
     <xacro:include filename="$(find fishbot_description)/urdf/fishbot/common_inertia.xacro"/>
     <xacro:macro name="laser_xacro" params="laser_name xyz rpy">
+    <!-- gazebo中添加颜色 -->
+    <gazebo reference="{laser_name}_cylinder_link">
+        <material>Gazebo/Gray</material>
+    </gazebo>
+    <gazebo reference="${laser_name}_link">
+        <material>Gazebo/Gray</material>
+    </gazebo>
         <!-- 雷达支撑杆 laser_cylinder_link -->
         <link name="${laser_name}_cylinder_link">
-            <visual name="laser_cylinder_visual">
+            <visual>
                 <origin xyz="0.0 0.0 0.0" rpy="0.0 0.0 0.0"/>
                 <geometry>
@@ -14,5 +21,5 @@
                 </material>
             </visual>
-            <collision name="laser_cylinder_collision">
+            <collision>
                 <origin xyz="0.0 0.0 0.0" rpy="0.0 0.0 0.0"/>
                 <geometry>
@@ -28,5 +35,5 @@
         <link name="${laser_name}_link">
         <!-- 部件的外观描述 -->
-            <visual name="laser_visual">
+            <visual>
             <!-- 沿着自己几何中心的偏移和旋转量 -->
                 <origin xyz="0.0 0.0 0.0" rpy="0.0 0.0 0.0"/>
@@ -39,5 +46,5 @@
             </visual>
             <!-- 碰撞属性 -->
-            <collision name="laser_collision">
+            <collision>
             <!-- 沿着自己几何中心的偏移和旋转量 -->
                 <origin xyz="0.0 0.0 0.0" rpy="0.0 0.0 0.0"/>
