Commit message: 第六章结束

File: chapt6/chapt6_ws/src/fishbot_description/urdf/fishbot/fishbot.urdf.xacro (robot description, xacro)
@@ -20,7 +20,9 @@
 <!-- Gazebo 插件 -->
 <xacro:include filename="$(find fishbot_description)/urdf/fishbot/plugins/gazebo_control_plugin.xacro" />
-<xacro:gazebo_control_plugin />
-<!-- <xacro:include filename="$(find fishbot_description)/urdf/fishbot/fishbot.ros2_control.xacro" /> -->
-<!-- <xacro:fishbot_ros2_control /> -->
+<xacro:include filename="$(find fishbot_description)/urdf/fishbot/plugins/gazebo_sensor_plugin.xacro" />
+<xacro:include filename="$(find fishbot_description)/urdf/fishbot/fishbot.ros2_control.xacro" />
+<!-- <xacro:gazebo_control_plugin /> -->
+<xacro:gazebo_sensor_plugin />
+<xacro:fishbot_ros2_control />
 </robot>
 <!-- ros2 launch fishbot_description display_robot.launch.py urdf_path:=/home/rick/ROS2_learn/chapt6/chapt6_ws/src/fishbot_description/urdf/fishbot/fishbot.urdf.xacro -->

File: chapt6/chapt6_ws/src/fishbot_description/urdf/fishbot/plugins/gazebo_sensor_plugin.xacro (robot description, xacro)
@@ -30,5 +30,5 @@
                     <range>
                         <min>0.120000</min>
-                        <max>8.0</max>
+                        <max>10.0</max>
                         <resolution>0.015000</resolution>
                     </range>

File: chapt6/chapt6_ws/src/fishbot_description/urdf/fishbot/sensor/camera.urdf.xacro (robot description, xacro)
@@ -32,4 +32,5 @@
             <xacro:box_inertia m="0.01" w="0.02" h="0.10" d="0.02" />
         </link>
+        <link name="${camera_name}_optical_link"></link>
         <!-- 机器人的关节，用于连接camera_link和base_link -->
         <joint name="${camera_name}_joint" type="fixed">
@@ -38,4 +39,9 @@
             <origin xyz="${xyz}" rpy="${rpy}"/>
         </joint>
+        <joint name="${camera_name}_optical_joint" type="fixed">
+            <parent link="${camera_name}_link"/>
+            <child link="${camera_name}_optical_link"/>
+            <origin xyz="0 0 0" rpy="${-pi/2} 0.0 ${-pi/2}"/>
+        </joint>
     </xacro:macro>
 </robot>
